File: hardware/v2/trigger/power.kicad_sch (KiCad schematic)
At the start: 20 parts, among them U1 LT3461A, U2 TPS7A4701, U3 TPS7A4701

Commit message: generate pdfs
Changed lines of the file:
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@@
 (kicad_sch
-	(version 20231120)
+	(version 20250114)
 	(generator "eeschema")
-	(generator_version "8.0")
+	(generator_version "9.0")
 	(paper "A4")
 	(title_block
