File: hardware/v2/trigger/trigger.kicad_sch (KiCad schematic)
At the start: 30 parts, among them J1 Conn_02x03_Top_Bottom, J10 Conn_Coaxial_Small, J11 Conn_Coaxial_Small, J12 Conn_02x03_Top_Bottom, J13 Conn_Coaxial_Small, J2 Conn_Coaxial_Small, J3 Conn_Coaxial_Small, J4 Conn_Coaxial_Small, J5 Conn_02x03_Top_Bottom, J6 Conn_Coaxial_Small, J7 Conn_Coaxial_Small, J8 Conn_Coaxial_Small, J9 Conn_02x03_Top_Bottom

Commit message: generate pdfs
Other:
- note added: "+5V +34.3V +3.4V +1.7V"
- note added: "AMPLIFIED ANALOG"
- note added: "INPUT - IN OUTPUT - BIAS - OPAMP - REF"
- note added: "SIPM - SENSL"
- note added: "x4"
Changed lines of the file:
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@@
 (kicad_sch
-	(version 20231120)
+	(version 20250114)
 	(generator "eeschema")
-	(generator_version "8.0")
+	(generator_version "9.0")
 	(paper "A4")
 	(title_block
@@
 		(comment 4 "Alex Xia")
 	)
+	(text "\nx4"
+		(exclude_from_sim no)
+		(at 108.204 64.262 0)
+		(effects
+			(font
+				(size 1.27 1.27)
+			)
+			(justify left)
+		)
+	)
+	(text "\n+5V\n\n\n+34.3V\n+3.4V\n+1.7V"
+		(exclude_from_sim no)
+		(at 71.374 69.342 0)
+		(effects
+			(font
+				(size 1.27 1.27)
+			)
+			(justify left)
+		)
+	)
+	(text "AMPLIFIED ANALOG"
+		(exclude_from_sim no)
+		(at 182.88 94.996 0)
+		(effects
+			(font
+				(size 1.27 1.27)
+			)
+		)
+	)
+	(text "SIPM\n- SENSL\n"
+		(exclude_from_sim no)
+		(at 97.282 64.262 0)
+		(effects
+			(font
+				(size 1.27 1.27)
+			)
+			(justify left)
+		)
+	)
+	(text "INPUT\n- IN\n\nOUTPUT\n- BIAS\n- OPAMP\n- REF\n"
+		(exclude_from_sim no)
+		(at 60.706 69.342 0)
+		(effects
+			(font
+				(size 1.27 1.27)
+			)
+			(justify left)
+		)
+	)
 	(junction
 		(at 203.2 137.16)
@@
 		(at 96.52 60.96)
 		(size 24.13 25.4)
+		(exclude_from_sim no)
+		(in_bom yes)
+		(on_board yes)
+		(dnp no)
 		(fields_autoplaced yes)
 		(stroke
@@
 		(at 130.81 60.96)
 		(size 35.56 25.4)
+		(exclude_from_sim no)
+		(in_bom yes)
+		(on_board yes)
+		(dnp no)
 		(fields_autoplaced yes)
 		(stroke
@@
 		(at 59.69 60.96)
 		(size 24.13 25.4)
+		(exclude_from_sim no)
+		(in_bom yes)
+		(on_board yes)
+		(dnp no)
 		(fields_autoplaced yes)
 		(stroke
@@
 		)
 	)
+	(embedded_fonts no)
 )
